File: PCB/Petri.kicad_pcb (KiCad board)
At the start: 2 copper layers, 160.8 x 120.7 mm, 18 parts, among them IC1 TMP236A4DBZR, IC2 REF3040AIDBZT, IC3 TLV7031DCKR, Q1 2N7002NXAKR, U1 12BH616P-GR

Commit message: Updated PCB
work completed:
- added proper dxf edge cuts from fusion file
- rerouted some tracks and positioned battery
to be done:
- position battery holder exactly at ½ height
- add cuts for case (staggered?)
Parts:
- moved R4 20.1 mm to (155.4, 129.5)
- moved C1 15.9 mm to (211.8, 118.6)
- moved C3 15.9 mm to (205.6, 118.6)
- moved C4 15.9 mm to (199.4, 119.6)
- moved C5 15.9 mm to (202.6, 116.2)
- moved IC1 15.9 mm to (189.8, 119.6)
- moved Q1 15.9 mm to (199.2, 115.2)
- moved R1 15.9 mm to (199.8, 122.2)
- moved R2 15.9 mm to (196.6, 121.2)
- moved C2 15.9 mm to (204.0, 121.0)
- moved D1 15.9 mm to (215.0, 115.8)
- moved IC2 15.9 mm to (208.6, 118.8)
- moved IC3 15.9 mm to (202.6, 118.8)
- moved R3 15.9 mm to (214.8, 117.8)
- moved R5 13.2 mm to (72.4, 125.7)
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Routing:
- net Net-(LED1-Pad2): track 169.4 -> 197.8 mm
- net Net-(R3-Pad2): track 88.7 -> 66.0 mm
- net Net-(LED1-Pad1): track 2.35 -> 13.8 mm
- net Net-(D1-Pad2): track 16.5 -> 27.4 mm
- net Net-(R4-Pad2): track 77.9 -> 83.3 mm
- net Net-(R5-Pad2): track 99.3 -> 94.6 mm
Other:
- board size 160.8 x 120.7 mm -> 160 x 120 mm
